File: hardware/nunchuk64/nunchuk64.sch (KiCad schematic (older format))
At the start: 28 parts, among them J1 DB9_Female, J2 DB9_Female, J3 Conn_02x03_Odd_Even, P1 CONN_WII, P2 CONN_WII, Q1 BSS138, Q2 BSS138, Q3 BSS138, Q4 BSS138, SW1 SW_Push, U1 AMS1117-3V3, U2 ATMEGA328P-AU

Commit message: Created fingers inside Connectors-Wii:CONN_WII for those hard to get connectors
Parts:
- P1, P2: footprint Connector_Wii:CONN_WII -> Connectors_WII:CONN_WII
Connections:
- no-connect marks 6 -> 4
Changed lines of the file:
@@
 F 0 "P1" H 2000 4400 60  0000 C CNN
 F 1 "CONN_WII" H 1800 4800 60  0000 C CNN
-F 2 "Connector_Wii:CONN_WII" H 1800 4300 60  0000 C CNN
+F 2 "Connectors_WII:CONN_WII" H 1800 4300 60  0000 C CNN
 F 3 "" H 1550 4600 60  0000 C CNN
 	1    1800 4600
@@
 F 0 "P2" H 2000 5950 60  0000 C CNN
 F 1 "CONN_WII" H 1800 6350 60  0000 C CNN
-F 2 "Connector_Wii:CONN_WII" H 1700 5850 60  0000 C CNN
+F 2 "Connectors_WII:CONN_WII" H 1700 5850 60  0000 C CNN
 F 3 "" H 1550 6150 60  0000 C CNN
 	1    1800 6150
@@
 Text Label 7100 4000 0    60   ~ 0
 SCL_
-NoConn ~ 2250 4600
-NoConn ~ 2250 6150
 $Comp
 L BSS138 Q3

Commit message: rounded corners. wii_conn_edge replaces old conn
Parts:
- P1, P2: footprint Connectors_WII:CONN_WII -> Connectors_WII:CONN_WII_EDGECON
Changed lines of the file:
@@
 F 0 "P1" H 2000 4400 60  0000 C CNN
 F 1 "CONN_WII" H 1800 4800 60  0000 C CNN
-F 2 "Connectors_WII:CONN_WII" H 1800 4300 60  0000 C CNN
+F 2 "Connectors_WII:CONN_WII_EDGECON" H 1800 4300 60  0000 C CNN
 F 3 "" H 1550 4600 60  0000 C CNN
 	1    1800 4600
@@
 F 0 "P2" H 2000 5950 60  0000 C CNN
 F 1 "CONN_WII" H 1800 6350 60  0000 C CNN
-F 2 "Connectors_WII:CONN_WII" H 1700 5850 60  0000 C CNN
+F 2 "Connectors_WII:CONN_WII_EDGECON" H 1700 5850 60  0000 C CNN
 F 3 "" H 1550 6150 60  0000 C CNN
 	1    1800 6150
